Commit message: fix(hero): repack go2/spot meshes with node transforms + textures, K1/spot colors, G1 greeting, dimmer lights, tall-screen hero cap
Co-Authored-By: Claude Sonnet 5.5 <noreply@anthropic.com>

File: public/models/spot.urdf (robot description, URDF)
Before this commit: robot spot, 26 links, 25 joints
Links:
- link base_arm_link: geometry collision mesh filename=base_link.stl scale=0.001 0.001 0.001; visual mesh filename=base_link.stl scale=0.001 0.001 0.001
- link finger: geometry collision mesh filename=finger.stl scale=0.001 0.001 0.001; visual mesh filename=finger.stl scale=0.001 0.001 0.001
- link gripper: geometry collision mesh filename=gripper.stl scale=0.001 0.001 0.001; visual mesh filename=gripper.stl scale=0.001 0.001 0.001
- link link1: geometry collision mesh filename=link1.stl scale=0.001 0.001 0.001; visual mesh filename=link1.stl scale=0.001 0.001 0.001
- link link2: geometry collision mesh filename=link2.stl scale=0.001 0.001 0.001; visual mesh filename=link2.stl scale=0.001 0.001 0.001
- link link3: geometry collision mesh filename=link3.stl scale=0.001 0.001 0.001; visual mesh filename=link3.stl scale=0.001 0.001 0.001
- link link4: geometry collision mesh filename=link4.stl scale=0.001 0.001 0.001; visual mesh filename=link4.stl scale=0.001 0.001 0.001
- link wrist: geometry collision mesh filename=wrist.stl scale=0.001 0.001 0.001; visual mesh filename=wrist.stl scale=0.001 0.001 0.001
