Commit message: feat(hero): add nova-carter, locobot, XLeRobot-style SO-101; ducks face viewer; publications before skills; tighten projects gap
Co-Authored-By: Claude Sonnet 5.5 <noreply@anthropic.com>

File: public/models/microduck.urdf (robot description, URDF)
Before this commit: robot microduck, 17 links, 16 joints
Links:
- link ankle_left: geometry visual mesh filename=ankle_left.stl scale=1.0 1.0 1.0; visual mesh filename=foot_left.stl scale=1.0 1.0 1.0
- link ankle_right: geometry visual mesh filename=ankle_right.stl scale=1.0 1.0 1.0; visual mesh filename=foot_right.stl scale=1.0 1.0 1.0
- link hip_left: geometry visual mesh filename=hip_l.stl scale=1.0 1.0 1.0; visual mesh filename=seeed_bearing__configuration__22x16x4.stl scale=1.0 1.0 1.0
- link hip_right: geometry visual mesh filename=hip_l.stl scale=1.0 1.0 1.0; visual mesh filename=seeed_bearing__configuration__22x16x4.stl scale=1.0 1.0 1.0
- link jaw: geometry visual mesh filename=jaw.stl scale=1.0 1.0 1.0; visual mesh filename=jaw_soft.stl scale=1.0 1.0 1.0
- link jaw_soft: geometry visual mesh filename=bottom_head_shell.stl scale=1.0 1.0 1.0; visual mesh filename=elec_rpi_robot_hat_pcb.stl scale=1.0 1.0 1.0
- link leg_left: geometry visual mesh filename=leg.stl scale=1.0 1.0 1.0; visual mesh filename=xl330.stl scale=1.0 1.0 1.0
- link leg_right: geometry visual mesh filename=leg.stl scale=1.0 1.0 1.0; visual mesh filename=xl330.stl scale=1.0 1.0 1.0
- link neck: geometry visual mesh filename=neck.stl scale=1.0 1.0 1.0; visual mesh filename=neck.stl scale=1.0 1.0 1.0
- link neck_pitch: geometry visual mesh filename=neck_pitch.stl scale=1.0 1.0 1.0; visual mesh filename=seeed_bearing__configuration__22x16x4.stl scale=1.0 1.0 1.0
- link trunk_base: geometry visual mesh filename=banana_pcb_locker.stl scale=1.0 1.0 1.0; visual mesh filename=left_shell.stl scale=1.0 1.0 1.0
- link upper_leg_left: geometry visual mesh filename=seeed_bearing__configuration__22x16x4.stl scale=1.0 1.0 1.0; visual mesh filename=upper_leg_left.stl scale=1.0 1.0 1.0
- link upper_leg_right: geometry visual mesh filename=seeed_bearing__configuration__22x16x4.stl scale=1.0 1.0 1.0; visual mesh filename=upper_leg_right.stl scale=1.0 1.0 1.0
- link yaw2roll_left: geometry visual mesh filename=bearing_roll.stl scale=1.0 1.0 1.0; visual mesh filename=seeed_bearing__configuration__22x16x4.stl scale=1.0 1.0 1.0
- link yaw2roll_right: geometry visual mesh filename=bearing_roll.stl scale=1.0 1.0 1.0; visual mesh filename=seeed_bearing__configuration__22x16x4.stl scale=1.0 1.0 1.0
- link yaw_roll_motion: geometry visual mesh filename=seeed_bearing__configuration__22x16x4.stl scale=1.0 1.0 1.0; visual mesh filename=seeed_bearing__configuration__22x16x4.stl scale=1.0 1.0 1.0
