Commit message: feat(hero): real LoCoBot Kobuki + XLeRobot URDFs, microduck somersault/roll, nova-carter to left
Co-Authored-By: Claude Sonnet 5.5 <noreply@anthropic.com>

File: docs/models/locobot.urdf (robot description, URDF)
Before this commit: robot locobot, 15 links, 13 joints
Links:
- removed link /ar_tag_link
- removed link /arm_base_link
- removed link /base_footprint
- removed link /ee_arm_link
- removed link /ee_gripper_link
- removed link /fingers_link
- removed link /forearm_link
- removed link /gripper_bar_link
- removed link /gripper_link
- removed link /gripper_prop_link
- removed link /left_finger_link
- removed link /right_finger_link
- removed link /shoulder_link
- removed link /upper_arm_link
- removed link /wrist_link
- added link locobot/ar_tag_link, mass 0.016507; collision mesh filename=mobile_wx200_10_ar_tag.stl scale=0.001 0.001 0.001; visual mesh filename=mobile_wx200_10_ar_tag.stl scale=0.001 0.001 0.001
- added link locobot/arm_base_link, mass 0.379673; collision mesh filename=mobile_wx200_1_base.stl scale=0.001 0.001 0.001; visual mesh filename=mobile_wx200_1_base.stl scale=0.001 0.001 0.001
- added link locobot/arm_cradle_link, mass 0.017626; collision mesh filename=locobot_arm_cradle.stl scale=0.001 0.001 0.001; visual mesh filename=locobot_arm_cradle.stl scale=0.001 0.001 0.001
- added link locobot/base_footprint
- added link locobot/base_link, mass 2.4; collision cylinder length=0.10938 radius=0.178; visual mesh filename=kobuki.dae
- added link locobot/battery_link, mass 1.194; collision mesh filename=locobot_battery.stl scale=0.001 0.001 0.001; visual mesh filename=locobot_battery.stl scale=0.001 0.001 0.001
- added link locobot/camera_depth_link
- added link locobot/camera_link, mass 0.072; collision mesh filename=locobot_camera.stl scale=0.001 0.001 0.001; visual mesh filename=locobot_camera.stl scale=0.001 0.001 0.001
- added link locobot/camera_tower_link, mass 2.282808; collision mesh filename=locobot_camera_tower_small_simple.stl scale=0.001 0.001 0.001; visual mesh filename=locobot_camera_tower_small.stl scale=0.001 0.001 0.001
- added link locobot/caster_back_link, mass 0.01; collision cylinder length=0.0176 radius=0.017
- added link locobot/caster_front_link, mass 0.01; collision cylinder length=0.0176 radius=0.017
- added link locobot/cliff_sensor_front_link, mass 0.0001
- added link locobot/cliff_sensor_left_link, mass 0.0001
- added link locobot/cliff_sensor_right_link, mass 0.0001
- added link locobot/ee_arm_link, mass 0.001
- added link locobot/ee_gripper_link, mass 0.001
- added link locobot/fingers_link, mass 0.001
- added link locobot/forearm_link, mass 0.283651; collision mesh filename=mobile_wx200_4_forearm.stl scale=0.001 0.001 0.001; visual mesh filename=mobile_wx200_4_forearm.stl scale=0.001 0.001 0.001
- added link locobot/gripper_bar_link, mass 0.034199; collision mesh filename=mobile_wx200_8_gripper_bar.stl scale=0.001 0.001 0.001; visual mesh filename=mobile_wx200_8_gripper_bar.stl scale=0.001 0.001 0.001
- added link locobot/gripper_link, mass 0.072885; collision mesh filename=mobile_wx200_6_gripper.stl scale=0.001 0.001 0.001; visual mesh filename=mobile_wx200_6_gripper.stl scale=0.001 0.001 0.001
- added link locobot/gripper_prop_link, mass 0.00434; collision mesh filename=mobile_wx200_7_gripper_prop.stl scale=0.001 0.001 0.001; visual mesh filename=mobile_wx200_7_gripper_prop.stl scale=0.001 0.001 0.001
- added link locobot/gyro_link, mass 0.001
- added link locobot/left_finger_link, mass 0.016246; collision mesh filename=mobile_wx200_9_gripper_finger.stl scale=0.001 0.001 0.001; visual mesh filename=mobile_wx200_9_gripper_finger.stl scale=0.001 0.001 0.001
- added link locobot/pan_link, mass 0.098997; collision mesh filename=locobot_pan.stl scale=0.001 0.001 0.001; visual mesh filename=locobot_pan.stl scale=0.001 0.001 0.001
- added link locobot/plate_link, mass 0.571995; collision mesh filename=locobot_base_plate.stl scale=0.001 0.001 0.001; visual mesh filename=locobot_base_plate.stl scale=0.001 0.001 0.001
- added link locobot/right_finger_link, mass 0.016246; collision mesh filename=mobile_wx200_9_gripper_finger.stl scale=0.001 0.001 0.001; visual mesh filename=mobile_wx200_9_gripper_finger.stl scale=0.001 0.001 0.001
- added link locobot/shoulder_link, mass 0.480879; collision mesh filename=mobile_wx200_2_shoulder.stl scale=0.001 0.001 0.001; visual mesh filename=mobile_wx200_2_shoulder.stl scale=0.001 0.001 0.001
- added link locobot/tilt_link, mass 0.019845; collision mesh filename=locobot_tilt.stl scale=0.001 0.001 0.001; visual mesh filename=locobot_tilt.stl scale=0.001 0.001 0.001
- added link locobot/upper_arm_link, mass 0.297781; collision mesh filename=mobile_wx200_3_upper_arm.stl scale=0.001 0.001 0.001; visual mesh filename=mobile_wx200_3_upper_arm.stl scale=0.001 0.001 0.001
- added link locobot/wheel_left_link, mass 0.01; collision cylinder length=0.0206 radius=0.0352; visual mesh filename=kobuki_wheel.dae
- added link locobot/wheel_right_link, mass 0.01; collision cylinder length=0.0206 radius=0.0350; visual mesh filename=kobuki_wheel.dae
- added link locobot/wrist_link, mass 0.084957; collision mesh filename=mobile_wx200_5_wrist.stl scale=0.001 0.001 0.001; visual mesh filename=mobile_wx200_5_wrist.stl scale=0.001 0.001 0.001
Joints:
- added joint arm_base_link_joint: type fixed, parent locobot/plate_link, child locobot/arm_base_link, origin xyz=0.097277 0 0.0095 rpy=0 0 0, axis 0 0 0
- added joint arm_cradle: type fixed, parent locobot/camera_tower_link, child locobot/arm_cradle_link, origin xyz=0.0215 0 0.1195 rpy=0 0 0, axis 0 0 0
- added joint base_joint: type fixed, parent locobot/base_footprint, child locobot/base_link, origin xyz=0 0 0.0102 rpy=0 0 0
- added joint battery: type fixed, parent locobot/plate_link, child locobot/battery_link, origin xyz=-0.007 0 0.0125 rpy=0 0 0
- added joint camera: type fixed, parent locobot/tilt_link, child locobot/camera_link, origin xyz=0.05318 0.0175 0.000009 rpy=0 0 0
- added joint camera_depth_joint: type fixed, parent locobot/camera_link, child locobot/camera_depth_link, origin xyz=0 0 0 rpy=-1.5707963267948966 0 -1.5707963267948966
- added joint camera_tower: type fixed, parent locobot/base_link, child locobot/camera_tower_link, origin xyz=-0.023997 -0.000044 0.08823 rpy=0 0 0
- added joint caster_back_joint: type fixed, parent locobot/base_link, child locobot/caster_back_link, origin xyz=-0.135 0.0 0.009 rpy=-1.57079632679 0 0
- added joint caster_front_joint: type fixed, parent locobot/base_link, child locobot/caster_front_link, origin xyz=0.115 0.0 0.007 rpy=-1.57079632679 0 0
- added joint cliff_sensor_front_joint: type fixed, parent locobot/base_link, child locobot/cliff_sensor_front_link, origin xyz=0.156 0.00 0.0214 rpy=0 1.57079632679 0
- added joint cliff_sensor_left_joint: type fixed, parent locobot/base_link, child locobot/cliff_sensor_left_link, origin xyz=0.08734 0.13601 0.0214 rpy=0 1.57079632679 0
- added joint cliff_sensor_right_joint: type fixed, parent locobot/base_link, child locobot/cliff_sensor_right_link, origin xyz=0.085 -0.13601 0.0214 rpy=0 1.57079632679 0
- added joint gyro_joint: type fixed, parent locobot/base_link, child locobot/gyro_link, origin xyz=0.056 0.062 0.0202 rpy=0 0 0
- added joint pan: type revolute, parent locobot/camera_tower_link, child locobot/pan_link, origin xyz=0.047228 0 0.38425 rpy=0 0 0, axis 0 0 1, limit lower=-1.5707963267948966 upper=1.5707963267948966 effort=2 velocity=3.141592653589793
- added joint plate: type fixed, parent locobot/base_link, child locobot/plate_link, origin xyz=0.0 0 0.08825 rpy=0 0 0
- added joint tilt: type revolute, parent locobot/pan_link, child locobot/tilt_link, origin xyz=0.025034 0 0.019 rpy=0 0 0, axis 0 1 0, limit lower=-1.5707963267948966 upper=1.3089969389957472 effort=2 velocity=3.141592653589793
- added joint wheel_left_joint: type continuous, parent locobot/base_link, child locobot/wheel_left_link, origin xyz=0.00 0.115 0.0250 rpy=-1.57079632679 0 0, axis 0 0 1
- added joint wheel_right_joint: type continuous, parent locobot/base_link, child locobot/wheel_right_link, origin xyz=0.00 -0.115 0.0250 rpy=-1.57079632679 0 0, axis 0 0 1
- joint ar_tag: child /ar_tag_link -> locobot/ar_tag_link; parent /ee_arm_link -> locobot/ee_arm_link
- joint ee_arm: child /ee_arm_link -> locobot/ee_arm_link; parent /gripper_link -> locobot/gripper_link
- joint ee_bar: child /fingers_link -> locobot/fingers_link; parent /gripper_bar_link -> locobot/gripper_bar_link
- joint ee_gripper: child /ee_gripper_link -> locobot/ee_gripper_link; parent /fingers_link -> locobot/fingers_link
- joint elbow: child /forearm_link -> locobot/forearm_link; parent /upper_arm_link -> locobot/upper_arm_link
- joint gripper: child /gripper_prop_link -> locobot/gripper_prop_link; parent /ee_arm_link -> locobot/ee_arm_link
- joint gripper_bar: child /gripper_bar_link -> locobot/gripper_bar_link; parent /ee_arm_link -> locobot/ee_arm_link
- joint left_finger: child /left_finger_link -> locobot/left_finger_link; parent /fingers_link -> locobot/fingers_link
- joint right_finger: child /right_finger_link -> locobot/right_finger_link; parent /fingers_link -> locobot/fingers_link
- joint shoulder: child /upper_arm_link -> locobot/upper_arm_link; parent /shoulder_link -> locobot/shoulder_link
- joint waist: child /shoulder_link -> locobot/shoulder_link; parent /arm_base_link -> locobot/arm_base_link
- joint wrist_angle: child /wrist_link -> locobot/wrist_link; parent /forearm_link -> locobot/forearm_link
- joint wrist_rotate: child /gripper_link -> locobot/gripper_link; parent /wrist_link -> locobot/wrist_link
